Commit message: Tried to change the model and failed

File: ros2_ws/src/MAMA_robot/urdf/robot.urdf (robot description, URDF)
Before this commit: robot MAMA_robot, 4 links, 3 joints
Links:
- removed link base_footprint
- removed link left_wheel
- removed link right_wheel
- link base_link: geometry collision mesh filename=package://MAMA_robot/meshes/model.stl scale=0.001 0.001 0.001; visual mesh filename=package://MAMA_robot/meshes/model.stl scale=0.001 0.001 0.001
Joints:
- removed joint base_joint
- removed joint left_wheel_joint
- removed joint right_wheel_joint

Commit message: robot bien exportado para video, falta añadir comportamiento

File: ros2_ws/src/MAMA_robot/urdf/robot.urdf (robot description, URDF)
Before this commit: robot MAMA_robot, 1 links, 0 joints
Links:
- added link base_footprint
- link base_link: geometry collision box size=0.32 0.40 0.50; visual mesh filename=package://MAMA_robot/meshes/model.stl scale=0.09 0.09 0.09
Joints:
- added joint base_joint: type fixed, parent base_footprint, child base_link, origin xyz=0 0 0 rpy=0 0 0
